File: mma8652_brkout.sch (KiCad schematic (older format))
At the start: 8 parts, among them U1 MMA8652

Commit message: - move mma8652 to kicadlib.
Parts:
- U1: footprint (none) -> ~
Changed lines of the file:
@@
 LIBS:contrib
 LIBS:valves
+LIBS:kicadlib
 LIBS:mma8652_brkout-cache
 EELAYER 27 0
@@
 Sheet 1 1
 Title ""
-Date "15 jan 2014"
+Date "16 jan 2014"
 Rev ""
 Comp ""
@@
 Comment4 ""
 $EndDescr
-$Comp
-L MMA8652 U1
-U 1 1 52D6E4A5
-P 5900 3300
-F 0 "U1" H 5900 2850 60  0000 C CNN
-F 1 "MMA8652" H 5900 3750 60  0000 C CNN
-F 2 "" H 5800 3200 60  0000 C CNN
-F 3 "" H 5800 3200 60  0000 C CNN
-	1    5900 3300
-	1    0    0    -1
-$EndComp
 $Comp
 L C C2
@@
 Text Notes 4350 5150 0    60   ~ 0
 http://www.mouser.com/ds/2/161/MMA8652FC-254149.pdf
+$Comp
+L MMA8652 U1
+U 1 1 52D73DD3
+P 5900 3300
+F 0 "U1" H 5900 2850 60  0000 C CNN
+F 1 "MMA8652" H 5900 3750 60  0000 C CNN
+F 2 "~" H 5800 3200 60  0000 C CNN
+F 3 "~" H 5800 3200 60  0000 C CNN
+	1    5900 3300
+	1    0    0    -1
+$EndComp
 $EndSCHEMATC

Commit message: - start pcb
Parts:
- added P1: VDD, ~, symbol TST
- added P2: GND, ~, symbol TST
- added P3: VDDIO, ~, symbol TST
- added P4: SCL, ~, symbol TST
- added P5: SDA, ~, symbol TST
- added P6: INT1, ~, symbol TST
- added P7: INT2, ~, symbol TST
Connections:
- net GND: now also P2.1
- net INT2: now also P7.1; no longer U1.3 (INT1)
- net SCL: now also P4.1
- net SDA: now also P5.1
- net VDD: now also P1.1
- net VDDIO: now also P3.1
- new net INT1: P6.1, U1.3 (INT1)
Changed lines of the file:
@@
 Sheet 1 1
 Title ""
-Date "16 jan 2014"
+Date "17 jan 2014"
 Rev ""
 Comp ""
@@
 Connection ~ 4550 3850
 Text GLabel 5150 3300 0    60   Input ~ 0
-INT2
+INT1
 Wire Wire Line
 	5150 3300 5250 3300
@@
 	1    0    0    -1
 $EndComp
+$Comp
+L TST P1
+U 1 1 52D88DCF
+P 1700 3150
+F 0 "P1" H 1700 3450 40  0000 C CNN
+F 1 "VDD" H 1700 3400 30  0000 C CNN
+F 2 "~" H 1700 3150 60  0000 C CNN
+F 3 "~" H 1700 3150 60  0000 C CNN
+	1    1700 3150
+	1    0    0    -1
+$EndComp
+Text GLabel 1700 3250 3    60   Input ~ 0
+VDD
+$Comp
+L TST P3
+U 1 1 52D88DDE
+P 2000 3150
+F 0 "P3" H 2000 3450 40  0000 C CNN
+F 1 "VDDIO" H 2000 3400 30  0000 C CNN
+F 2 "~" H 2000 3150 60  0000 C CNN
+F 3 "~" H 2000 3150 60  0000 C CNN
+	1    2000 3150
+	1    0    0    -1
+$EndComp
+Text GLabel 2000 3250 3    60   Input ~ 0
+VDDIO
+$Comp
+L GND #PWR07
+U 1 1 52D88DFF
+P 1850 3250
+F 0 "#PWR07" H 1850 3250 30  0001 C CNN
+F 1 "GND" H 1850 3180 30  0001 C CNN
+F 2 "" H 1850 3250 60  0000 C CNN
+F 3 "" H 1850 3250 60  0000 C CNN
+	1    1850 3250
+	1    0    0    -1
+$EndComp
+$Comp
+L TST P2
+U 1 1 52D88E11
+P 1850 3150
+F 0 "P2" H 1850 3450 40  0000 C CNN
+F 1 "GND" H 1850 3400 30  0000 C CNN
+F 2 "~" H 1850 3150 60  0000 C CNN
+F 3 "~" H 1850 3150 60  0000 C CNN
+	1    1850 3150
+	1    0    0    -1
+$EndComp
+Wire Wire Line
+	1700 3150 1700 3250
+Wire Wire Line
+	1850 3250 1850 3150
+Wire Wire Line
+	2000 3150 2000 3250
+Text GLabel 2150 3250 3    60   Input ~ 0
+SCL
+Text GLabel 2300 3250 3    60   Input ~ 0
+SDA
+Text GLabel 2450 3250 3    60   Input ~ 0
+INT1
+Text GLabel 2600 3250 3    60   Input ~ 0
+INT2
+$Comp
+L TST P4
+U 1 1 52D88EDB
+P 2150 3150
+F 0 "P4" H 2150 3450 40  0000 C CNN
+F 1 "SCL" H 2150 3400 30  0000 C CNN
+F 2 "~" H 2150 3150 60  0000 C CNN
+F 3 "~" H 2150 3150 60  0000 C CNN
+	1    2150 3150
+	1    0    0    -1
+$EndComp
+$Comp
+L TST P5
+U 1 1 52D88EE1
+P 2300 3150
+F 0 "P5" H 2300 3450 40  0000 C CNN
+F 1 "SDA" H 2300 3400 30  0000 C CNN
+F 2 "~" H 2300 3150 60  0000 C CNN
+F 3 "~" H 2300 3150 60  0000 C CNN
+	1    2300 3150
+	1    0    0    -1
+$EndComp
+$Comp
+L TST P6
+U 1 1 52D88EE7
+P 2450 3150
+F 0 "P6" H 2450 3450 40  0000 C CNN
+F 1 "INT1" H 2450 3400 30  0000 C CNN
+F 2 "~" H 2450 3150 60  0000 C CNN
+F 3 "~" H 2450 3150 60  0000 C CNN
+	1    2450 3150
+	1    0    0    -1
+$EndComp
+$Comp
+L TST P7
+U 1 1 52D88EED
+P 2600 3150
+F 0 "P7" H 2600 3450 40  0000 C CNN
+F 1 "INT2" H 2600 3400 30  0000 C CNN
+F 2 "~" H 2600 3150 60  0000 C CNN
+F 3 "~" H 2600 3150 60  0000 C CNN
+	1    2600 3150
+	1    0    0    -1
+$EndComp
+Wire Wire Line
+	2150 3150 2150 3250
+Wire Wire Line
+	2300 3250 2300 3150
+Wire Wire Line
+	2450 3150 2450 3250
+Wire Wire Line
+	2600 3150 2600 3250
 $EndSCHEMATC
