File: mma8652_brkout.kicad_pcb (KiCad board)
At the start: 2 copper layers, 0 parts

Commit message: - start pcb
Parts:
- added C1: 1uF, SM0603, F.Cu at (197.1, 55.4)
- added C2: 0.1uF, SM0603, F.Cu at (198.1, 51.3)
- added C3: 100nF, SM0603, F.Cu at (201.4, 57.4)
- added C4: 0.1uF, SM0603, F.Cu at (205.7, 53.6)
- added JP1: JUMPER, jmp_small, F.Cu at (192.8, 50.8)
- added P1: VDD, TEST_0.100, F.Cu at (177.8, 38.1)
- added P2: GND, TEST_0.100, F.Cu at (180.3, 38.1)
- added P3: VDDIO, TEST_0.100, F.Cu at (182.9, 38.1)
- added P4: SCL, TEST_0.100, F.Cu at (185.4, 38.1)
- added P5: SDA, TEST_0.100, F.Cu at (188.0, 38.1)
- added P6: INT1, TEST_0.100, F.Cu at (193.0, 38.1)
- added P7: INT2, TEST_0.100, F.Cu at (190.5, 38.1)
- added R1: 1K, SM0603, F.Cu at (190.2, 56.9)
- added R2: 1K, SM0603, F.Cu at (197.9, 58.9)
- added U1: MMA8652, mma8652, F.Cu at (185.2, 51.6)

Commit message: - more pcb
Parts:
- moved C4 27.5 mm to (179.8, 44.5), turned to 90 degrees
- moved R2 21.6 mm to (181.9, 44.5), turned to 90 degrees
- moved C3 19.1 mm to (185.4, 47.0), turned to 180 degrees
- moved JP1 16.3 mm to (177.8, 44.5)
- moved R1 12.5 mm to (189.7, 44.5), turned to 270 degrees
- moved C1 11.4 mm to (193.8, 44.5), turned to 270 degrees
- moved C2 9.35 mm to (191.8, 44.5), turned to 270 degrees
- moved U1 7.12 mm to (185.4, 44.5), turned to 180 degrees

Commit message: - save pcb. should be rev 0.1
Parts:
- moved R2 6.01 mm to (187.7, 45.8)
- moved C3 3.02 mm to (182.6, 45.8), turned to 270 degrees
- moved P6 2.54 mm to (190.5, 38.1)
- moved P7 2.54 mm to (193.0, 38.1)
- moved U1 0.64 mm to (185.4, 43.8), turned to 270 degrees
- moved R1 0.13 mm to (189.9, 44.5)
Routing:
- net VDD: track 0.00 -> 26.6 mm, vias 0 -> 4
- net VDDIO: track 0.00 -> 22.5 mm
- net SCL: track 0.00 -> 13.3 mm, vias 0 -> 2
- net INT2: track 0.00 -> 11.5 mm, vias 0 -> 1
- net SDA: track 0.00 -> 9.28 mm, vias 0 -> 2
- net INT1: track 0.00 -> 7.91 mm, vias 0 -> 1
- net N-000002: track 0.00 -> 3.76 mm
- added copper zone on B.Cu, net GND
- added copper zone on F.Cu, net GND
Other:
- board outline added: 19.1 x 11.4 mm
- net class Default: clearance 0.254 -> 0.1524
- rule trace_clearance: 0.254 -> 0.1524
- rule via_min_drill: 0.508 -> 0.3302
- rule via_min_size: 0.889 -> 0.5334
- board text added: "MMA8652 Breakout git.io/SH6DBg v 0.1 jan-2014"
